File: kicad/spinac_od_davida/tem-l3a/tem-l3a.sch (KiCad schematic (older format))
At the start: 11 parts, among them SW1 SW_Push, SW2 SW_Push, U1 LM555xM

Commit message: vývody
Parts:
- added J1: Conn_01x02_Male, symbol Connector:Conn_01x02_Male
- gave numbers to parts that had none: 2
- renumbered C1 to C2, R2 to R3, R3 to R4, SW2 to SW1, SW1 to SW2
Connections:
- net at C1.2, C2.2, D1.1 (K)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: now also J1.2 (Pin_2)
- net at R1.1, R3.1, RV1.1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: now also J1.1 (Pin_1)
Changed lines of the file:
@@
 $EndComp
 $Comp
-L Switch:SW_Push SW2
+L Switch:SW_Push SW1
 U 1 1 618B8F0E
 P 4750 4450
-F 0 "SW2" H 4750 4735 50  0000 C CNN
+F 0 "SW1" H 4750 4735 50  0000 C CNN
 F 1 "SW_Push" H 4750 4644 50  0000 C CNN
 F 2 "" H 4750 4650 50  0001 C CNN
@@
 $EndComp
 $Comp
-L Device:CP C1
+L Device:CP C2
 U 1 1 618BA883
 P 6950 4450
-F 0 "C1" H 7068 4496 50  0000 L CNN
+F 0 "C2" H 7068 4496 50  0000 L CNN
 F 1 "CP" H 7068 4405 50  0000 L CNN
 F 2 "" H 6988 4300 50  0001 C CNN
@@
 $EndComp
 $Comp
-L Device:R_Small R3
+L Device:R_Small R4
 U 1 1 618BD2C7
 P 8300 3950
-F 0 "R3" H 8359 3996 50  0000 L CNN
+F 0 "R4" H 8359 3996 50  0000 L CNN
 F 1 "R_Small" H 8359 3905 50  0000 L CNN
 F 2 "" H 8300 3950 50  0001 C CNN
@@
 $EndComp
 $Comp
-L Switch:SW_Push SW1
+L Switch:SW_Push SW2
 U 1 1 618BDABF
 P 7800 4450
-F 0 "SW1" H 7800 4735 50  0000 C CNN
+F 0 "SW2" H 7800 4735 50  0000 C CNN
 F 1 "SW_Push" H 7800 4644 50  0000 C CNN
 F 2 "" H 7800 4650 50  0001 C CNN
@@
 $EndComp
 $Comp
-L Device:C C?
+L Device:C C1
 U 1 1 618BF49D
 P 5150 4300
-F 0 "C?" H 5265 4346 50  0000 L CNN
+F 0 "C1" H 5265 4346 50  0000 L CNN
 F 1 "C" H 5265 4255 50  0000 L CNN
 F 2 "" H 5188 4150 50  0001 C CNN
@@
 	8300 3600 6600 3600
 $Comp
-L Device:R_Small R2
+L Device:R_Small R3
 U 1 1 618BD1DF
 P 7800 3250
-F 0 "R2" H 7859 3296 50  0000 L CNN
+F 0 "R3" H 7859 3296 50  0000 L CNN
 F 1 "R_Small" H 7859 3205 50  0000 L CNN
 F 2 "" H 7800 3250 50  0001 C CNN
@@
 Connection ~ 7800 4250
 $Comp
-L Device:R_Small R?
+L Device:R_Small R2
 U 1 1 618CC1EB
 P 6950 3200
-F 0 "R?" H 7009 3246 50  0000 L CNN
+F 0 "R2" H 7009 3246 50  0000 L CNN
 F 1 "R_Small" H 7009 3155 50  0000 L CNN
 F 2 "" H 6950 3200 50  0001 C CNN
@@
 Connection ~ 6100 2500
 $Comp
-L power:PWR_FLAG #FLG?
+L power:PWR_FLAG #FLG01
 U 1 1 618D1DE5
 P 3400 3950
-F 0 "#FLG?" H 3400 4025 50  0001 C CNN
+F 0 "#FLG01" H 3400 4025 50  0001 C CNN
 F 1 "PWR_FLAG" H 3400 4123 50  0000 C CNN
 F 2 "" H 3400 3950 50  0001 C CNN
@@
 $EndComp
 $Comp
-L power:PWR_FLAG #FLG?
+L power:PWR_FLAG #FLG02
 U 1 1 618D20CC
 P 3400 4250
-F 0 "#FLG?" H 3400 4325 50  0001 C CNN
+F 0 "#FLG02" H 3400 4325 50  0001 C CNN
 F 1 "PWR_FLAG" H 3400 4423 50  0000 C CNN
 F 2 "" H 3400 4250 50  0001 C CNN
@@
 	4000 4750 4750 4750
 Connection ~ 4750 4750
+$Comp
+L Connector:Conn_01x02_Male J1
+U 1 1 619E5037
+P 3050 4050
+F 0 "J1" H 3158 4231 50  0000 C CNN
+F 1 "Conn_01x02_Male" H 3158 4140 50  0000 C CNN
+F 2 "" H 3050 4050 50  0001 C CNN
+F 3 "~" H 3050 4050 50  0001 C CNN
+	1    3050 4050
+	1    0    0    -1
+$EndComp
+Wire Wire Line
+	3400 3950 3250 3950
+Wire Wire Line
+	3250 3950 3250 4050
+Connection ~ 3400 3950
+Wire Wire Line
+	3250 4150 3250 4250
+Wire Wire Line
+	3250 4250 3400 4250
+Connection ~ 3400 4250
 $EndSCHEMATC
