File: kicad/spinac_od_toma/tem-l3a.sch (KiCad schematic (older format))
At the start: 12 parts, among them J1 Conn_01x02_Male, SW1 SW_Push, SW2 SW_Push, U1 LM555xM

Commit message: Updated Toms file
Parts:
- added H1, H2: MountingHole, MountingHole:MountingHole_3.2mm_M3, symbol Mechanical:MountingHole
- C1: renamed from C2; value CP -> 100uF; footprint (none) -> Capacitor_THT:CP_Radial_D8.0mm_P5.00mm
- C2: renamed from C1; value C -> 100nF; footprint (none) -> Capacitor_SMD:C_0603_1608Metric
- D1: footprint (none) -> LED_SMD:LED_0603_1608Metric
- J1: footprint (none) -> Connector_PinHeader_2.54mm:PinHeader_1x02_P2.54mm_Vertical
- R1: value R_Small -> 10k; footprint (none) -> Resistor_SMD:R_0603_1608Metric_Pad1.05x0.95mm_HandSolder
- R2: renamed from R3; value R_Small -> 10k; footprint (none) -> Resistor_SMD:R_0603_1608Metric_Pad1.05x0.95mm_HandSolder
- R3: renamed from R4; value R_Small -> 470; footprint (none) -> Resistor_SMD:R_0603_1608Metric_Pad1.05x0.95mm_HandSolder
- R4: renamed from R2; value R_Small -> 10k; footprint (none) -> Resistor_SMD:R_0603_1608Metric_Pad1.05x0.95mm_HandSolder
- RV1: value R_POT -> 1M; footprint (none) -> Potentiometer_SMD:Potentiometer_ACP_CA14-VSMD_Vertical
- SW1, SW2: footprint (none) -> Button_Switch_SMD:Panasonic_EVQPUJ_EVQPUA
Connections:
- wire segments 48 -> 50
Other:
- moved on the sheet: C2
Changed lines of the file:
@@
 F 0 "SW1" H 4750 4735 50  0000 C CNN
 F 1 "SW_Push" H 4750 4644 50  0000 C CNN
-F 2 "" H 4750 4650 50  0001 C CNN
+F 2 "Button_Switch_SMD:Panasonic_EVQPUJ_EVQPUA" H 4750 4650 50  0001 C CNN
 F 3 "~" H 4750 4650 50  0001 C CNN
 	1    4750 4450
@@
 P 4750 3200
 F 0 "R1" H 4809 3246 50  0000 L CNN
-F 1 "R_Small" H 4809 3155 50  0000 L CNN
-F 2 "" H 4750 3200 50  0001 C CNN
+F 1 "10k" H 4809 3155 50  0000 L CNN
+F 2 "Resistor_SMD:R_0603_1608Metric_Pad1.05x0.95mm_HandSolder" H 4750 3200 50  0001 C CNN
 F 3 "~" H 4750 3200 50  0001 C CNN
 	1    4750 3200
@@
 $EndComp
 $Comp
-L Device:CP C2
+L Device:CP C1
 U 1 1 618BA883
 P 6950 4450
-F 0 "C2" H 7068 4496 50  0000 L CNN
-F 1 "CP" H 7068 4405 50  0000 L CNN
-F 2 "" H 6988 4300 50  0001 C CNN
+F 0 "C1" H 7068 4496 50  0000 L CNN
+F 1 "100uF" H 7068 4405 50  0000 L CNN
+F 2 "Capacitor_THT:CP_Radial_D8.0mm_P5.00mm" H 6988 4300 50  0001 C CNN
 F 3 "~" H 6950 4450 50  0001 C CNN
 	1    6950 4450
@@
 F 0 "D1" H 8293 4667 50  0000 C CNN
 F 1 "LED" H 8293 4576 50  0000 C CNN
-F 2 "" H 8300 4450 50  0001 C CNN
+F 2 "LED_SMD:LED_0603_1608Metric" H 8300 4450 50  0001 C CNN
 F 3 "~" H 8300 4450 50  0001 C CNN
 	1    8300 4450
@@
 $EndComp
 $Comp
-L Device:R_Small R4
+L Device:R_Small R3
 U 1 1 618BD2C7
 P 8300 3950
-F 0 "R4" H 8359 3996 50  0000 L CNN
-F 1 "R_Small" H 8359 3905 50  0000 L CNN
-F 2 "" H 8300 3950 50  0001 C CNN
+F 0 "R3" H 8359 3996 50  0000 L CNN
+F 1 "470" H 8359 3905 50  0000 L CNN
+F 2 "Resistor_SMD:R_0603_1608Metric_Pad1.05x0.95mm_HandSolder" H 8300 3950 50  0001 C CNN
 F 3 "~" H 8300 3950 50  0001 C CNN
 	1    8300 3950
@@
 F 0 "SW2" H 7800 4735 50  0000 C CNN
 F 1 "SW_Push" H 7800 4644 50  0000 C CNN
-F 2 "" H 7800 4650 50  0001 C CNN
+F 2 "Button_Switch_SMD:Panasonic_EVQPUJ_EVQPUA" H 7800 4650 50  0001 C CNN
 F 3 "~" H 7800 4650 50  0001 C CNN
 	1    7800 4450
@@
 P 6950 2800
 F 0 "RV1" H 6881 2846 50  0000 R CNN
-F 1 "R_POT" H 6881 2755 50  0000 R CNN
-F 2 "" H 6950 2800 50  0001 C CNN
+F 1 "1M" H 6881 2755 50  0000 R CNN
+F 2 "Potentiometer_SMD:Potentiometer_ACP_CA14-VSMD_Vertical" H 6950 2800 50  0001 C CNN
 F 3 "~" H 6950 2800 50  0001 C CNN
 	1    6950 2800
@@
 $EndComp
 $Comp
-L Device:C C1
+L Device:C C2
 U 1 1 618BF49D
-P 5150 4300
-F 0 "C1" H 5265 4346 50  0000 L CNN
-F 1 "C" H 5265 4255 50  0000 L CNN
-F 2 "" H 5188 4150 50  0001 C CNN
-F 3 "~" H 5150 4300 50  0001 C CNN
-	1    5150 4300
+P 5150 4350
+F 0 "C2" H 5265 4396 50  0000 L CNN
+F 1 "100nF" H 5265 4305 50  0000 L CNN
+F 2 "Capacitor_SMD:C_0603_1608Metric" H 5188 4200 50  0001 C CNN
+F 3 "~" H 5150 4350 50  0001 C CNN
+	1    5150 4350
 	1    0    0    -1
 $EndComp
@@
 	5600 3800 5150 3800
 Wire Wire Line
-	5150 3800 5150 4150
-Wire Wire Line
-	5150 4450 5150 4750
-Wire Wire Line
-	5150 4750 6100 4750
+	5150 4450 5150 4500
 Wire Wire Line
 	6100 4750 6100 4200
@@
 	8300 3600 6600 3600
 $Comp
-L Device:R_Small R3
+L Device:R_Small R2
 U 1 1 618BD1DF
 P 7800 3250
-F 0 "R3" H 7859 3296 50  0000 L CNN
-F 1 "R_Small" H 7859 3205 50  0000 L CNN
-F 2 "" H 7800 3250 50  0001 C CNN
+F 0 "R2" H 7859 3296 50  0000 L CNN
+F 1 "10k" H 7859 3205 50  0000 L CNN
+F 2 "Resistor_SMD:R_0603_1608Metric_Pad1.05x0.95mm_HandSolder" H 7800 3250 50  0001 C CNN
 F 3 "~" H 7800 3250 50  0001 C CNN
 	1    7800 3250
@@
 Connection ~ 7800 4250
 $Comp
-L Device:R_Small R2
+L Device:R_Small R4
 U 1 1 618CC1EB
 P 6950 3200
-F 0 "R2" H 7009 3246 50  0000 L CNN
-F 1 "R_Small" H 7009 3155 50  0000 L CNN
-F 2 "" H 6950 3200 50  0001 C CNN
+F 0 "R4" H 7009 3246 50  0000 L CNN
+F 1 "10k" H 7009 3155 50  0000 L CNN
+F 2 "Resistor_SMD:R_0603_1608Metric_Pad1.05x0.95mm_HandSolder" H 6950 3200 50  0001 C CNN
 F 3 "~" H 6950 3200 50  0001 C CNN
 	1    6950 3200
@@
 	4750 4650 4750 4750
 Wire Wire Line
-	4750 4750 5150 4750
-Connection ~ 5150 4750
-Wire Wire Line
 	4750 3600 4750 3300
 Connection ~ 4750 3600
@@
 Connection ~ 6100 2500
 $Comp
-L power:PWR_FLAG #FLG01
+L power:PWR_FLAG #FLG0101
 U 1 1 618D1DE5
 P 3400 3950
-F 0 "#FLG01" H 3400 4025 50  0001 C CNN
+F 0 "#FLG0101" H 3400 4025 50  0001 C CNN
 F 1 "PWR_FLAG" H 3400 4123 50  0000 C CNN
 F 2 "" H 3400 3950 50  0001 C CNN
@@
 $EndComp
 $Comp
-L power:PWR_FLAG #FLG02
+L power:PWR_FLAG #FLG0102
 U 1 1 618D20CC
 P 3400 4250
-F 0 "#FLG02" H 3400 4325 50  0001 C CNN
+F 0 "#FLG0102" H 3400 4325 50  0001 C CNN
 F 1 "PWR_FLAG" H 3400 4423 50  0000 C CNN
 F 2 "" H 3400 4250 50  0001 C CNN
@@
 	4000 4750 4750 4750
 Connection ~ 4750 4750
+Wire Wire Line
+	4750 4750 5150 4750
+Connection ~ 5150 4750
+Wire Wire Line
+	5150 4750 6100 4750
+Connection ~ 5150 4500
+Wire Wire Line
+	5150 4500 5150 4750
+Wire Wire Line
+	5150 3800 5150 4200
+Connection ~ 5150 4200
+Wire Wire Line
+	5150 4200 5150 4250
 $Comp
 L Connector:Conn_01x02_Male J1
-U 1 1 619E5037
-P 3050 4050
-F 0 "J1" H 3158 4231 50  0000 C CNN
-F 1 "Conn_01x02_Male" H 3158 4140 50  0000 C CNN
-F 2 "" H 3050 4050 50  0001 C CNN
-F 3 "~" H 3050 4050 50  0001 C CNN
-	1    3050 4050
-	1    0    0    -1
-$EndComp
-Wire Wire Line
-	3400 3950 3250 3950
-Wire Wire Line
-	3250 3950 3250 4050
+U 1 1 619F90F1
+P 2850 4000
+F 0 "J1" H 2958 4181 50  0000 C CNN
+F 1 "Conn_01x02_Male" H 2958 4090 50  0000 C CNN
+F 2 "Connector_PinHeader_2.54mm:PinHeader_1x02_P2.54mm_Vertical" H 2850 4000 50  0001 C CNN
+F 3 "~" H 2850 4000 50  0001 C CNN
+	1    2850 4000
+	1    0    0    -1
+$EndComp
+Wire Wire Line
+	3400 3950 3050 3950
+Wire Wire Line
+	3050 3950 3050 4000
 Connection ~ 3400 3950
 Wire Wire Line
-	3250 4150 3250 4250
-Wire Wire Line
-	3250 4250 3400 4250
+	3400 4250 3050 4250
+Wire Wire Line
+	3050 4250 3050 4100
 Connection ~ 3400 4250
+$Comp
+L Mechanical:MountingHole H1
+U 1 1 619FCFC1
+P 3550 2400
+F 0 "H1" H 3650 2446 50  0000 L CNN
+F 1 "MountingHole" H 3650 2355 50  0000 L CNN
+F 2 "MountingHole:MountingHole_3.2mm_M3" H 3550 2400 50  0001 C CNN
+F 3 "~" H 3550 2400 50  0001 C CNN
+	1    3550 2400
+	1    0    0    -1
+$EndComp
+$Comp
+L Mechanical:MountingHole H2
+U 1 1 619FD524
+P 8600 4950
+F 0 "H2" H 8700 4996 50  0000 L CNN
+F 1 "MountingHole" H 8700 4905 50  0000 L CNN
+F 2 "MountingHole:MountingHole_3.2mm_M3" H 8600 4950 50  0001 C CNN
+F 3 "~" H 8600 4950 50  0001 C CNN
+	1    8600 4950
+	1    0    0    -1
+$EndComp
 $EndSCHEMATC
