File: kicad/spinac_od_toma/tem-l3a.kicad_sch (KiCad schematic)
At the start: 14 parts, among them J1 Conn_01x02_Male, SW1 SW_Push, SW2 SW_Push, U1 LM555xM

Commit message: lul
Parts:
- C2: CLSC (none) -> C307331
- R1, R2, R4: CLSC (none) -> C25744
Changed lines of the file:
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@@
+      (effects (font (size 1.27 1.27)) hide)
+    )
+    (property "CLSC" "C25744" (id 4) (at 120.65 81.28 0)
       (effects (font (size 1.27 1.27)) hide)
     )
@@
     )
     (property "Datasheet" "~" (id 3) (at 198.12 82.55 0)
+      (effects (font (size 1.27 1.27)) hide)
+    )
+    (property "CLSC" "C25744" (id 4) (at 198.12 82.55 0)
       (effects (font (size 1.27 1.27)) hide)
     )
@@
       (effects (font (size 1.27 1.27)) hide)
     )
+    (property "CLSC" "C307331" (id 4) (at 130.81 110.49 0)
+      (effects (font (size 1.27 1.27)) hide)
+    )
     (pin "1")
     (pin "2")
@@
       (effects (font (size 1.27 1.27)) hide)
     )
+    (property "CLSC" "C25744" (id 4) (at 176.53 81.28 0)
+      (effects (font (size 1.27 1.27)) hide)
+    )
